Commit message: pegs

File: objects/peg.urdf.xacro (robot description, xacro)
@@ -1,8 +1,8 @@
 <?xml version="1.0"?>
-<robot name="peg">
-  <link name="peg_link">
+<robot name="$(arg name)" xmlns:xacro="http://www.ros.org/wiki/xacro">
+  <link name="$(arg name)/peg_link">
     <visual>
       <geometry>
-        <cylinder length="0.4" radius="0.05"/>
+        <cylinder length="0.4" radius="0.03"/>
       </geometry>
       <material name="whitish">
@@ -10,6 +10,18 @@
       </material>
     </visual>
+    <collision>
+      <geometry>
+        <cylinder length="0.4" radius="0.03"/>
+      </geometry>
+    </collision>
   </link>
-  <link name="base_link">
+  <link name="$(arg name)/base_link">
+    <inertial>
+      <mass value="30" />
+      <inertia
+        ixx="1" ixy="0"   ixz="0"
+                iyy="1"   iyz="0"
+                          izz="1" />
+    </inertial>
     <visual>
       <geometry>
@@ -20,14 +32,20 @@
       </material>
     </visual>
+    <collision>
+      <geometry>
+        <box size="0.6 0.6 0.1"/>
+      </geometry>
+    </collision>
    </link>
-  <joint name="base_to_peg" type="fixed">
-    <parent link="base_link"/>
-    <child link="peg_link"/>
+  <joint name="$(arg name)/base_to_peg" type="fixed">
+    <parent link="$(arg name)/base_link"/>
+    <child link="$(arg name)/peg_link"/>
     <origin xyz="0.0 0.0 0.25"/>
   </joint>
-  <!--<joint name="$(arg prefix)/base_to_world" type="fixed">
+  <link name="world"/>
+  <joint name="$(arg name)/base_to_world" type="fixed">
     <parent link="world"/>
-    <child link="$(arg prefix)/base_link"/>
-    <origin xyz="$(arg xx) $(arg yy) 0.05"/>
+    <child link="$(arg name)/base_link"/>
+    <origin xyz="$(arg xx) $(arg yy) 0.07"/>
   </joint>
 </robot>
