Commit message: changes to square components: added gazebo tags

File: objects/construct_common.urdf.xacro (robot description, xacro)
@@ -8,4 +8,15 @@
   <xacro:property name="edge_joint_offset" value="0.04" />
   <xacro:property name="edge_joint_y_offset" value="0.15" />
+  <xacro:property name="corner_mass" value="0.25"/>
+  <xacro:property name="edge_mass" value="0.28"/>
+  <xacro:macro name="cs_gz_ref" params="prefix id">
+    <gazebo reference="${prefix}/${id}">
+      <material>Gazebo/WoodPallet</material>
+      <selfCollide>true</selfCollide>
+      <gravity>true</gravity>
+      <mu1>0.80</mu1>
+      <mu2>0.80</mu2>
+    </gazebo>
+  </xacro:macro>
   <!--
     Macro for definition of a construction object corner cube.
@@ -17,9 +28,9 @@
     <link name="${prefix}/${id}">
       <inertial>
-        <mass value="0.2" />
+        <mass value="${corner_mass}" />
         <inertia
-          ixx="1" ixy="0"   ixz="0"
-                  iyy="1"   iyz="0"
-                  izz="1" />
+          ixx="0.0012" ixy="0"   ixz="0"
+                  iyy="0.0012"   iyz="0"
+                  izz="0.0012" />
       </inertial>
       <visual>
@@ -37,4 +48,5 @@
       </collision>
     </link>
+    <xacro:cs_gz_ref prefix="${prefix}" id="${id}" />
     <xacro:if value="true">
       <joint name="${prefix}/cs_${id}_${child1_id}" type="floating">
@@ -58,9 +70,9 @@
     <link name="${prefix}/${id}">
       <inertial>
-        <mass value="0.2" />
+        <mass value="${corner_mass}" />
         <inertia
-          ixx="1" ixy="0"   ixz="0"
-                  iyy="1"   iyz="0"
-                  izz="1" />
+          ixx="0.0012" ixy="0"   ixz="0"
+                  iyy="0.0012"   iyz="0"
+                  izz="0.0012" />
       </inertial>
       <visual>
@@ -78,4 +90,5 @@
       </collision>
     </link>
+    <xacro:cs_gz_ref prefix="${prefix}" id="${id}" />
     <xacro:if value="true">
       <joint name="${prefix}/cs_${id}_${child1_id}" type="floating">
@@ -90,9 +103,9 @@
     <link name="${prefix}/${id}">
       <inertial>
-        <mass value="0.2" />
+        <mass value="${corner_mass}" />
         <inertia
-          ixx="1" ixy="0"   ixz="0"
-                  iyy="1"   iyz="0"
-                  izz="1" />
+          ixx="0.0012" ixy="0"   ixz="0"
+                  iyy="0.0012"   iyz="0"
+                  izz="0.0012" />
       </inertial>
       <visual>
@@ -110,4 +123,5 @@
       </collision>
     </link>
+    <xacro:cs_gz_ref prefix="${prefix}" id="${id}" />
   </xacro:macro>
   <!--
@@ -120,9 +134,9 @@
     <link name="${prefix}/${id}">
       <inertial>
-        <mass value="0.22" />
+        <mass value="${edge_mass}" />
         <inertia
-          ixx="1" ixy="0"   ixz="0"
-                  iyy="1"   iyz="0"
-                  izz="1" />
+          ixx="0.0012" ixy="0"   ixz="0"
+                  iyy="0.0012"   iyz="0"
+                  izz="0.0012" />
       </inertial>
       <visual>
@@ -140,4 +154,5 @@
       </collision>
     </link>
+    <xacro:cs_gz_ref prefix="${prefix}" id="${id}" />
     <xacro:if value="true">
       <joint name="${prefix}/cs_${id}_${child_id}" type="floating">
@@ -157,9 +172,9 @@
     <link name="${prefix}/${id}">
       <inertial>
-        <mass value="0.22" />
+        <mass value="${edge_mass}" />
         <inertia
-          ixx="1" ixy="0"   ixz="0"
-                  iyy="1"   iyz="0"
-                  izz="1" />
+          ixx="0.0012" ixy="0"   ixz="0"
+                  iyy="0.0012"   iyz="0"
+                  izz="0.0012" />
       </inertial>
       <visual>
@@ -177,4 +192,5 @@
       </collision>
     </link>
+    <xacro:cs_gz_ref prefix="${prefix}" id="${id}" />
   </xacro:macro>
 </robot>

Commit message: changes to square, launch file: gazebo integration

File: objects/construct_common.urdf.xacro (robot description, xacro)
@@ -2,9 +2,9 @@
 <robot xmlns:xacro="http://www.ros.org/wiki/xacro">
   <xacro:property name="PI" value="3.1415926535897931" />
-  <xacro:property name="corner_width" value="0.10" />
-  <xacro:property name="corner_joint_offset" value="0.05" />
-  <xacro:property name="edge_width" value="0.08" />
+  <xacro:property name="corner_width" value="0.08" />
+  <xacro:property name="corner_joint_offset" value="0.04" />
+  <xacro:property name="edge_width" value="0.06" />
   <xacro:property name="edge_length" value="0.30" />
-  <xacro:property name="edge_joint_offset" value="0.04" />
+  <xacro:property name="edge_joint_offset" value="0.03" />
   <xacro:property name="edge_joint_y_offset" value="0.15" />
   <xacro:property name="corner_mass" value="0.25"/>

File: objects/construct_square.urdf.xacro (robot description, xacro)
@@ -1,4 +1,11 @@
 <robot name="$(arg name)" xmlns:xacro="http://www.ros.org/wiki/xacro">
   <xacro:include filename="$(find lcsr_spacenav)/objects/construct_common.urdf.xacro"/>
+  <!-- root link to the world frame -->
+  <link name="world" />
+  <joint name="world_to_$(arg name)" type="floating">
+    <origin xyz="$(arg xyz)" rpy="$(arg rpy)"/>
+    <parent link="world"/>
+    <child link="$(arg name)/corner1"/>
+  </joint>
   <xacro:cs_corner_1child prefix="$(arg name)"
     id="corner1"

Commit message: joints must be continuous to read them into the plug in

File: objects/construct_common.urdf.xacro (robot description, xacro)
@@ -50,5 +50,5 @@
     <xacro:cs_gz_ref prefix="${prefix}" id="${id}" />
     <xacro:if value="true">
-      <joint name="${prefix}/cs_${id}_${child1_id}" type="floating">
+      <joint name="${prefix}/cs_${id}_${child1_id}" type="continuous">
         <parent link="${prefix}/${id}"/>
         <child link="${prefix}/${child1_id}"/>
@@ -58,5 +58,5 @@
     </xacro:if>
     <xacro:if value="true">
-      <joint name="${prefix}/cs_${id}_${child2_id}" type="floating">
+      <joint name="${prefix}/cs_${id}_${child2_id}" type="continuous">
         <parent link="${prefix}/${id}"/>
         <child link="${prefix}/${child2_id}"/>
@@ -92,5 +92,5 @@
     <xacro:cs_gz_ref prefix="${prefix}" id="${id}" />
     <xacro:if value="true">
-      <joint name="${prefix}/cs_${id}_${child1_id}" type="floating">
+      <joint name="${prefix}/cs_${id}_${child1_id}" type="continuous">
         <parent link="${prefix}/${id}"/>
         <child link="${prefix}/${child1_id}"/>
@@ -156,5 +156,5 @@
     <xacro:cs_gz_ref prefix="${prefix}" id="${id}" />
     <xacro:if value="true">
-      <joint name="${prefix}/cs_${id}_${child_id}" type="floating">
+      <joint name="${prefix}/cs_${id}_${child_id}" type="continuous">
         <parent link="${prefix}/${id}"/>
         <child link="${prefix}/${child_id}"/>

File: objects/construct_square.urdf.xacro (robot description, xacro)
@@ -64,5 +64,5 @@
     <namespace>observed</namespace>
     <reference_frame>/world</reference_frame>
-    <verbosity>3</verbosity>
+    <verbosity>1</verbosity>
   </plugin>
   <!--<plugin name="gazebo_tutorials" filename="libgazebo_tutorials.so"/>-->

Commit message: less joint mobility

File: objects/construct_common.urdf.xacro (robot description, xacro)
@@ -50,17 +50,19 @@
     <xacro:cs_gz_ref prefix="${prefix}" id="${id}" />
     <xacro:if value="true">
-      <joint name="${prefix}/cs_${id}_${child1_id}" type="continuous">
+      <joint name="${prefix}/cs_${id}_${child1_id}" type="revolute">
         <parent link="${prefix}/${id}"/>
         <child link="${prefix}/${child1_id}"/>
         <origin xyz="${corner_joint_offset} ${corner_joint_offset} ${corner_joint_offset}"
           rpy="0 0 0"/>
-      </joint>
-    </xacro:if>
-    <xacro:if value="true">
-      <joint name="${prefix}/cs_${id}_${child2_id}" type="continuous">
+        <limit effort="30" velocity="0.0" lower="-0.01" upper="0.01" />
+      </joint>
+    </xacro:if>
+    <xacro:if value="true">
+      <joint name="${prefix}/cs_${id}_${child2_id}" type="revolute">
         <parent link="${prefix}/${id}"/>
         <child link="${prefix}/${child2_id}"/>
         <origin xyz="${corner_joint_offset} ${-1*corner_joint_offset} ${corner_joint_offset}"
           rpy="0 0 ${PI}"/>
+        <limit effort="30" velocity="0.0" lower="-0.01" upper="0.01" />
       </joint>
     </xacro:if>
@@ -92,8 +94,9 @@
     <xacro:cs_gz_ref prefix="${prefix}" id="${id}" />
     <xacro:if value="true">
-      <joint name="${prefix}/cs_${id}_${child1_id}" type="continuous">
+      <joint name="${prefix}/cs_${id}_${child1_id}" type="revolute">
         <parent link="${prefix}/${id}"/>
         <child link="${prefix}/${child1_id}"/>
         <origin xyz="${xyz}" rpy="${rpy}"/>
+        <limit effort="30" velocity="0.0" lower="-0.01" upper="0.01" />
       </joint>
     </xacro:if>
@@ -156,8 +159,9 @@
     <xacro:cs_gz_ref prefix="${prefix}" id="${id}" />
     <xacro:if value="true">
-      <joint name="${prefix}/cs_${id}_${child_id}" type="continuous">
+      <joint name="${prefix}/cs_${id}_${child_id}" type="revolute">
         <parent link="${prefix}/${id}"/>
         <child link="${prefix}/${child_id}"/>
         <origin xyz="${xyz}" rpy="${rpy}"/>
+        <limit effort="30" velocity="0.0" lower="-0.01" upper="0.01" />
       </joint>
     </xacro:if>

File: objects/construct_square.urdf.xacro (robot description, xacro)
@@ -60,4 +60,6 @@
       <enable_latch>1</enable_latch>
       <latch_strength>30.0</latch_strength>
+      <latch_distance>0.05</latch_distance>
+      <latch_rotation>1.05</latch_rotation>
       <updates_per_second>180.0</updates_per_second>
     </plugin>

Commit message: settings for building objects -- color, plugin config, etc.

File: objects/construct_common.urdf.xacro (robot description, xacro)
@@ -19,4 +19,11 @@
     </gazebo>
   </xacro:macro>
+  <xacro:macro name="gz_joint_settings" params="joint_ref">
+    <gazebo reference="${joint_ref}">
+      <physics>
+        <provide_feedback>true</provide_feedback>
+      </physics>
+    </gazebo>
+  </xacro:macro>
   <!--
     Macro for definition of a construction object corner cube.
@@ -39,5 +46,5 @@
         </geometry>
         <material name="cs_dark">
-          <color rgba="0.5 0.5 0.5 1"/>
+          <color rgba="0.5 0.3 0.1 1"/>
         </material>
       </visual>
@@ -57,4 +64,5 @@
         <limit effort="30" velocity="0.0" lower="-0.01" upper="0.01" />
       </joint>
+      <xacro:gz_joint_settings joint_ref="${prefix}/cs_${id}_${child1_id}" />
     </xacro:if>
     <xacro:if value="true">
@@ -66,4 +74,5 @@
         <limit effort="30" velocity="0.0" lower="-0.01" upper="0.01" />
       </joint>
+      <xacro:gz_joint_settings joint_ref="${prefix}/cs_${id}_${child2_id}" />
     </xacro:if>
   </xacro:macro>
@@ -83,5 +92,5 @@
         </geometry>
         <material name="cs_dark">
-          <color rgba="0.5 0.5 0.5 1"/>
+          <color rgba="0.5 0.3 0.1 1"/>
         </material>
       </visual>
@@ -100,4 +109,5 @@
         <limit effort="30" velocity="0.0" lower="-0.01" upper="0.01" />
       </joint>
+      <xacro:gz_joint_settings joint_ref="${prefix}/cs_${id}_${child1_id}" />
     </xacro:if>
   </xacro:macro>
@@ -117,5 +127,5 @@
         </geometry>
         <material name="cs_dark">
-          <color rgba="0.5 0.5 0.5 1"/>
+          <color rgba="0.5 0.3 0.1 1"/>
         </material>
       </visual>
@@ -148,5 +158,5 @@
         </geometry>
         <material name="cs_grey">
-          <color rgba="0.7 0.7 0.7 1"/>
+          <color rgba="0.7 0.5 0.3 1"/>
         </material>
       </visual>
@@ -165,4 +175,5 @@
         <limit effort="30" velocity="0.0" lower="-0.01" upper="0.01" />
       </joint>
+      <xacro:gz_joint_settings joint_ref="${prefix}/cs_${id}_${child_id}" />
     </xacro:if>
   </xacro:macro>
@@ -187,5 +198,5 @@
         </geometry>
         <material name="cs_grey">
-          <color rgba="0.7 0.7 0.7 1"/>
+          <color rgba="0.7 0.5 0.3 1"/>
         </material>
       </visual>

File: objects/construct_square.urdf.xacro (robot description, xacro)
@@ -59,5 +59,6 @@
       <verbosity>2</verbosity>
       <enable_latch>1</enable_latch>
-      <latch_strength>30.0</latch_strength>
+      <latch_torque>0.0</latch_torque>
+      <latch_force>15.0</latch_force>
       <latch_distance>0.05</latch_distance>
       <latch_rotation>1.05</latch_rotation>
