Commit message: fixed package ref in ring urdf

File: objects/ring.urdf.xacro (robot description, xacro)
@@ -20,5 +20,5 @@
       <origin rpy="0 0 0 " xyz="0 0 0"/>
       <geometry>
-        <mesh filename="package://lcsr_spacenav/objects/ring.dae"/>
+        <mesh filename="package://lcsr_collab/objects/ring.dae"/>
       </geometry>
     </visual>
@@ -26,5 +26,5 @@
       <origin rpy="0 0 0 " xyz="0 0 0"/>
       <geometry>
-        <mesh filename="package://lcsr_spacenav/objects/ring.stl"/>
+        <mesh filename="package://lcsr_collab/objects/ring.stl"/>
       </geometry>
     </collision>

Commit message: tests to see if there is a better way to handle rings in MoveIt, added a srdf.xacro file. xacro file may or may not actually be compatible with the robot right now.

File: objects/ring.urdf.xacro (robot description, xacro)
@@ -1,10 +1,13 @@
 <robot name="$(arg name)"
   xmlns:xacro="http://www.ros.org/wiki/xacro">
-  <!--<link name="world"/>-->
-  <!-- Fix this robot to the world -->
-  <!--<joint name="world_joint"  type="floating">
-    <origin xyz="0 0 0" rpy="0 0 0" />
+  <!-- Attach this robot to the world:
+    - this was changed because of the way MoveIt works
+    - we need to determine the relationship between any object and the world
+  -->
+  <!--<link name="world"/>
+  <joint name="$(arg name)_to_world"  type="floating">
+    <origin xyz="$(arg xx) $(arg yy) $(arg zz)" rpy="0 0 0" />
     <parent link="world"/>
-    <child link="ring_link"/>
+    <child link="$(arg name)/ring_link"/>
   </joint>-->
   <link name = "$(arg name)/ring_link">
