Commit message: changes to collab files to fix package names

File: collab_env/objects/construct_square.urdf.xacro (robot description, xacro)
@@ -1,4 +1,4 @@
 <robot name="$(arg name)" xmlns:xacro="http://www.ros.org/wiki/xacro">
-  <xacro:include filename="$(find lcsr_collab)/objects/construct_common.urdf.xacro"/>
+  <xacro:include filename="$(find collab_env)/objects/construct_common.urdf.xacro"/>
   <!-- root link to the world frame -->
   <!--<link name="world" />
@@ -54,5 +54,5 @@
   />
   <gazebo>
-    <plugin name="lcsr_construction_plugin" filename="liblcsr_construction_plugin.so" >
+    <plugin name="collab_construction_plugin" filename="libcollab_construction_plugin.so" >
       <namespace>/observed</namespace>
       <reference_frame>/world</reference_frame>

File: collab_env/objects/ring.urdf.xacro (robot description, xacro)
@@ -23,5 +23,5 @@
       <origin rpy="0 0 0 " xyz="0 0 0"/>
       <geometry>
-        <mesh filename="package://lcsr_collab/objects/ring.dae"/>
+        <mesh filename="package://collab_env/objects/ring.dae"/>
       </geometry>
     </visual>
@@ -29,10 +29,10 @@
       <origin rpy="0 0 0 " xyz="0 0 0"/>
       <geometry>
-        <mesh filename="package://lcsr_collab/objects/ring.stl"/>
+        <mesh filename="package://collab_env/objects/ring.stl"/>
       </geometry>
     </collision>
   </link>
   <gazebo>
-    <plugin name="lcsr_construction_plugin" filename="liblcsr_construction_plugin.so" >
+    <plugin name="collab_construction_plugin" filename="libcollab_construction_plugin.so" >
       <namespace></namespace>
       <reference_frame>/world</reference_frame>
