Commit message: made the peg bases a bit smaller to make the planning problem easier, at least for now

File: collab_env/objects/peg.urdf.xacro (robot description, xacro)
@@ -26,5 +26,5 @@
     <visual>
       <geometry>
-        <box size="0.6 0.6 0.1"/>
+        <box size="0.3 0.3 0.1"/>
       </geometry>
       <material name="whitish">
@@ -34,5 +34,5 @@
     <collision>
       <geometry>
-        <box size="0.6 0.6 0.1"/>
+        <box size="0.3 0.3 0.1"/>
       </geometry>
     </collision>

Commit message: added a frame for the top of the peg

File: collab_env/objects/peg.urdf.xacro (robot description, xacro)
@@ -1,4 +1,11 @@
 <?xml version="1.0"?>
 <robot name="$(arg name)" xmlns:xacro="http://www.ros.org/wiki/xacro">
+  <link name="$(arg name)/peg_top_link">
+  </link>
+  <joint name="$(arg name)/peg_to_top" type="fixed">
+    <parent link="$(arg name)/peg_link"/>
+    <child link="$(arg name)/peg_top_link"/>
+    <origin xyz="0.0 0.0 0.2"/>
+  </joint>
   <link name="$(arg name)/peg_link">
     <visual>
