Commit message: fixed up srdf to create new semantic arm descriptions

File: collab_env/sim/model/wam_7dof_arm.srdf.xacro (robot description, xacro)
@@ -2,58 +2,58 @@
 <robot xmlns:xacro="http://www.ros.org/wiki/xacro">
   <xacro:macro name="wam_7dof_arm" params="arm_name prefix">
-    <group name="arm">
-        <joint name="$(arg prefix)/base_yaw_joint" />
-        <joint name="$(arg prefix)/shoulder_pitch_joint" />
-        <joint name="$(arg prefix)/shoulder_yaw_joint" />
-        <joint name="$(arg prefix)/elbow_pitch_joint" />
-        <joint name="$(arg prefix)/wrist_yaw_joint" />
-        <joint name="$(arg prefix)/wrist_pitch_joint" />
-        <joint name="$(arg prefix)/palm_yaw_joint" />
+    <group name="${arm_name}">
+      <joint name="${prefix}/base_yaw_joint" />
+      <joint name="${prefix}/shoulder_pitch_joint" />
+      <joint name="${prefix}/shoulder_yaw_joint" />
+      <joint name="${prefix}/elbow_pitch_joint" />
+      <joint name="${prefix}/wrist_yaw_joint" />
+      <joint name="${prefix}/wrist_pitch_joint" />
+      <joint name="${prefix}/palm_yaw_joint" />
     </group>
-    <!--GROUP STATES: Purpose: Define a named state for a particular group, in terms of joint values. This is useful to define states like 'folded arms'-->
-    <group_state name="zero" group="arm">
-        <joint name="$(arg prefix)/base_yaw_joint" value="0" />
-        <joint name="$(arg prefix)/elbow_pitch_joint" value="0" />
-        <joint name="$(arg prefix)/palm_yaw_joint" value="0" />
-        <joint name="$(arg prefix)/shoulder_pitch_joint" value="0" />
-        <joint name="$(arg prefix)/shoulder_yaw_joint" value="0" />
-        <joint name="$(arg prefix)/wrist_pitch_joint" value="0" />
-        <joint name="$(arg prefix)/wrist_yaw_joint" value="0" />
+    <!--GROUP STATES: Purpose: Define a named state for a particular group, in terms of joint values. This is useful to define states like 'folded ${arm_name}s'-->
+    <group_state name="zero" group="${arm_name}">
+      <joint name="${prefix}/base_yaw_joint" value="0" />
+      <joint name="${prefix}/elbow_pitch_joint" value="0" />
+      <joint name="${prefix}/palm_yaw_joint" value="0" />
+      <joint name="${prefix}/shoulder_pitch_joint" value="0" />
+      <joint name="${prefix}/shoulder_yaw_joint" value="0" />
+      <joint name="${prefix}/wrist_pitch_joint" value="0" />
+      <joint name="${prefix}/wrist_yaw_joint" value="0" />
     </group_state>
-    <group_state name="cal" group="arm">
-        <joint name="$(arg prefix)/base_yaw_joint" value="0" />
-        <joint name="$(arg prefix)/elbow_pitch_joint" value="3.1415" />
-        <joint name="$(arg prefix)/palm_yaw_joint" value="0" />
-        <joint name="$(arg prefix)/shoulder_pitch_joint" value="-1.5707" />
-        <joint name="$(arg prefix)/shoulder_yaw_joint" value="0" />
-        <joint name="$(arg prefix)/wrist_pitch_joint" value="-1.5707" />
-        <joint name="$(arg prefix)/wrist_yaw_joint" value="0" />
-      </group_state>
-      <disable_collisions link1="$(arg prefix)/base_link" link2="$(arg prefix)/upper_arm_link"
-        reason="Adjacent" />
-      <disable_collisions link1="$(arg prefix)/hand/bhand_palm_link" link2="$(arg prefix)/hand/finger_1/prox_link"
-        reason="Adjacent" />
-      <disable_collisions link1="$(arg prefix)/hand/bhand_palm_link" link2="$(arg prefix)/hand/finger_2/prox_link"
-        reason="Adjacent" />
-      <disable_collisions link1="$(arg prefix)/hand/bhand_palm_link" link2="$(arg prefix)/wrist_pitch_link"
-        reason="Adjacent" />
-      <disable_collisions link1="$(arg prefix)/hand/bhand_palm_link" link2="$(arg prefix)/wrist_yaw_link"
-        reason="Adjacent" />
-      <disable_collisions link1="$(arg prefix)/hand/finger_1/dist_link" link2="$(arg prefix)/hand/finger_1/med_link"
-        reason="Adjacent" />
-      <disable_collisions link1="$(arg prefix)/hand/finger_2/dist_link" link2="$(arg prefix)/hand/finger_2/med_link"
-        reason="Adjacent" />
-      <disable_collisions link1="$(arg prefix)/hand/finger_3/dist_link" link2="$(arg prefix)/hand/finger_3/med_link"
-        reason="Adjacent" />
-      <disable_collisions link1="$(arg prefix)/shoulder_pitch_link" link2="$(arg prefix)/shoulder_yaw_link"
-        reason="Adjacent" />
-      <disable_collisions link1="$(arg prefix)/shoulder_pitch_link" link2="$(arg prefix)/upper_arm_link"
-        reason="Adjacent" />
-      <disable_collisions link1="$(arg prefix)/shoulder_yaw_link" link2="$(arg prefix)/upper_arm_link"
-        reason="Adjacent" />
-      <disable_collisions link1="$(arg prefix)/wrist_pitch_link" link2="$(arg prefix)/wrist_yaw_link"
-        reason="Adjacent" />
+    <group_state name="cal" group="${arm_name}">
+      <joint name="${prefix}/base_yaw_joint" value="0" />
+      <joint name="${prefix}/elbow_pitch_joint" value="3.1415" />
+      <joint name="${prefix}/palm_yaw_joint" value="0" />
+      <joint name="${prefix}/shoulder_pitch_joint" value="-1.5707" />
+      <joint name="${prefix}/shoulder_yaw_joint" value="0" />
+      <joint name="${prefix}/wrist_pitch_joint" value="-1.5707" />
+      <joint name="${prefix}/wrist_yaw_joint" value="0" />
+    </group_state>
+    <disable_collisions link1="${prefix}/base_link" link2="${prefix}/upper_${arm_name}_link"
+      reason="Adjacent" />
+    <disable_collisions link1="${prefix}/hand/bhand_palm_link" link2="${prefix}/hand/finger_1/prox_link"
+      reason="Adjacent" />
+    <disable_collisions link1="${prefix}/hand/bhand_palm_link" link2="${prefix}/hand/finger_2/prox_link"
+      reason="Adjacent" />
+    <disable_collisions link1="${prefix}/hand/bhand_palm_link" link2="${prefix}/wrist_pitch_link"
+      reason="Adjacent" />
+    <disable_collisions link1="${prefix}/hand/bhand_palm_link" link2="${prefix}/wrist_yaw_link"
+      reason="Adjacent" />
+    <disable_collisions link1="${prefix}/hand/finger_1/dist_link" link2="${prefix}/hand/finger_1/med_link"
+      reason="Adjacent" />
+    <disable_collisions link1="${prefix}/hand/finger_2/dist_link" link2="${prefix}/hand/finger_2/med_link"
+      reason="Adjacent" />
+    <disable_collisions link1="${prefix}/hand/finger_3/dist_link" link2="${prefix}/hand/finger_3/med_link"
+      reason="Adjacent" />
+    <disable_collisions link1="${prefix}/shoulder_pitch_link" link2="${prefix}/shoulder_yaw_link"
+      reason="Adjacent" />
+    <disable_collisions link1="${prefix}/shoulder_pitch_link" link2="${prefix}/upper_${arm_name}_link"
+      reason="Adjacent" />
+    <disable_collisions link1="${prefix}/shoulder_yaw_link" link2="${prefix}/upper_${arm_name}_link"
+      reason="Adjacent" />
+    <disable_collisions link1="${prefix}/wrist_pitch_link" link2="${prefix}/wrist_yaw_link"
+      reason="Adjacent" />
     <!--END EFFECTOR: Purpose: Represent information about an end effector.-->
-    <end_effector name="wrist_mount" parent_link="$(arg prefix)/wrist_palm_link" group="arm" />
+    <end_effector name="${prefix}/wrist_mount" parent_link="${prefix}/wrist_palm_link" group="${arm_name}" />
   </xacro:macro>
 </robot>
